File: frodo_io_module.kicad_sch (KiCad schematic)
At the start: 40 parts, among them J1 Conn_01x04_Pin, J1 Molex MicroFit 2x3, J2 Molex MicroFit 2x3, J4 Conn_01x04_Pin, SW1 SW_DIP_x06, U1 AZ1117H-ADJ, U1 STM32F072RBT6, U3 AZ1117-3.3, U5 AZ1117-5.0, Y1 8MHz

Commit message: cleanup/commenting for better readability, minor corrections
Parts:
- added R4: 1k, symbol Device:R
- J1: value Conn_01x04_Pin -> SWD Header
- J4: value Conn_01x04_Pin -> JST-GH 4Pin
- R3, R5: value 1000 -> 1k
- Y1: value 8MHz -> 8MHz 12pF
Connections:
- net VCC is gone; now on net +3.3V: SW1.10, SW1.11, SW1.7, SW1.8, SW1.9
- net GND: now also J2.1 (Pin_1)
- net HSE_IN: now also C11.1, Y1.3; no longer C10.1, Y1.1
- net HSE_OUT: now also R4.1; no longer C11.1, Y1.3
- net VCOM: now also SW1.12; no longer SW1.1
- net VSwitch renamed SW0
- net SW0: now also SW1.1; no longer SW1.12
- new net: C10.1, R4.2, Y1.1
Other:
- sheet DIP Switch2 renamed Digital Output
- removed sheet DIP Switch
- removed sheet DIP Switch1
- removed sheet DIP Switch3
- sheet Digital Output: file untitled.kicad_sch -> digital_output.kicad_sch
- note added: "3.3V Regulator"
- note added: "3.3V/5V Regulator for AIn/Com IOs"
- note added: "5V Regulator"
- note added: "AIn/Com IO Connectors"
- note added: "Digital Outputs"
- note added: "MCU"
- note added: "ModID DIP Switches"
- moved on the sheet: C1, C10, C11, C12, C13, C2, C3, C4, C5, C6, C7, C8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

Commit message: Add flash, CAN transceiver, 5V regulators, power filtering; minor corrections
Parts:
- removed C12: 10u, symbol Device:C
- removed C13: 22u, symbol Device:C
- removed U5: AZ1117-5.0, symbol Regulator_Linear:AZ1117-5.0
- added C12 (x4): 10u, symbol Device:C
- added C23, C24, C29: 1u, symbol Device:C
- added C25, C26, C27, C28, C30, C31, C32, C33, C34: 22u, symbol Device:C
- added C43 (x3): 100n, Capacitor_SMD:C_0402_1005Metric_Pad0.74x0.62mm_HandSolder, symbol Device:C_Small
- added D1, D2: D_Schottky, symbol Device:D_Schottky
- added D3, D4, D5, D6: LED, symbol Device:LED
- added F1, F2: 10A, symbol Device:Fuse
- added JP1, JP2: +VSW_Sel, symbol Jumper:SolderJumper_2_Open
- added JP3, JP4: VDC_Sel, symbol Jumper:SolderJumper_2_Open
- added JP5, JP6: Vext_Sel, symbol Jumper:SolderJumper_2_Open
- added JP7, JP8: +5V_Sel, symbol Jumper:SolderJumper_2_Open
- added R35, R36, R38: 220, symbol Device:R
- added R37: 680, symbol Device:R
- added R39: 120, DNP, symbol Device:R_Small
- added R40: 100, symbol Device:R
- added U4: W25Q128JVP, Package_SO:SOIC-8_5.275x5.275mm_P1.27mm, symbol frodo_io_module:W25Q128JVP
- added U5: MCP2562-E-SN, Package_SO:SOIC-8_3.9x4.9mm_P1.27mm, symbol Interface_CAN_LIN:MCP2562-E-SN
- added U6, U7: L7805, symbol Regulator_Linear:L7805
- J1: value SWD Header -> SWD
- R1: value 500 -> 680
- R3: value 1k -> 820
Connections:
- net +3.3V: now also C43.2, C43.2, R35.1, R36.1, R38.1, U4.8 (VCC), U5.5 (Vio)
- net +5V: now also C43.2, D1.1 (K), D2.1 (K), JP7.1 (A), JP8.1 (A), R37.1, U5.3 (VDD)
- net +VSW: now also C12.1, C12.1, F1.1, JP1.1 (A), JP2.1 (A), U6.1 (IN), U7.1 (IN)
- net CAN+: now also R39.1, U5.7 (CANH)
- net CAN-: now also R39.2, U5.6 (CANL)
- net GND: now also C12.2, C12.2, C12.2, C12.2, C23.2, C24.2, C25.2, C26.2, C27.2, C28.2, C29.2, C30.2, C31.2, C32.2, C33.2, C34.2, C43.1, C43.1, C43.1, D3.1 (K), R40.2, U4.4 (GND), U5.2 (VSS), U5.8 (STBY), U6.2 (GND), U7.2 (GND); no longer R5.2
- net VDC: now also F2.1, JP3.1 (A), JP4.1 (A)
- net SPI_CS_FLASH: now reaches U1.20 (PA4)
- net SPI_CS_FLASH: now also U4.1 (~{CS})
- net SPI1_SCK: now reaches U1.21 (PA5)
- net SPI1_SCK: now also U4.6 (CLK)
- net SPI1_MISO: now reaches U1.22 (PA6)
- net SPI1_MISO: now also U4.2 (DO(IO1))
- net SPI1_MOSI: now reaches U1.23 (PA7)
- net SPI1_MOSI: now also U4.5 (DI(IO0))
- net STAT_LED0: now reaches U1.40 (PC9)
- net STAT_LED0: now also D4.1 (K)
- net CAN_RX: now reaches U1.44 (PA11)
- net CAN_RX: now also U5.4 (RXD)
- net CAN_TX: now reaches U1.45 (PA12)
- net CAN_TX: now also U5.1 (TXD)
- net STAT_LED1: now reaches U1.51 (PC10)
- net STAT_LED1: now also D5.1 (K)
- net STAT_LED2: now reaches U1.52 (PC11)
- net STAT_LED2: now also D6.1 (K)
- new net: C23.1, C24.1, C25.1, C26.1, C27.1, C28.1, C33.1, C34.1, F1.2
- new net: D6.2 (A), R38.2
- new net: C29.1, C30.1, C31.1, C32.1, F2.2
- new net: R40.1, R5.2
- new net: D5.2 (A), R36.2
- new net: C12.1, D2.2 (A), U7.3 (OUT)
- new net: D4.2 (A), R35.2
- new net: D3.2 (A), R37.2
- new net: C12.1, D1.2 (A), U6.3 (OUT)
- new net Vboost: JP5.1 (A), JP6.1 (A)
- new net Vdrive: JP1.2 (B), JP2.2 (B), JP3.2 (B), JP4.2 (B), JP5.2 (B), JP6.2 (B), JP7.2 (B), JP8.2 (B)
- no-connect marks 24 -> 19
Other:
- note added: "5V Regulators"
- note added: "CAN Transceiver"
- note added: "Digital Output Voltage Select"
- note added: "Flash"
- note added: "Use high current schottky diodes with low voltage drop"
- note removed: "5V Regulator"
- moved on the sheet: C1, C10, C11, C12, C13, C2, C3, C4, C5, C6, C7, C8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
