File: frodo_io_module.kicad_sch (KiCad schematic)
At the start: 129 parts, among them J1 Molex MicroFit 2x3, J1 SWD, J2 Molex MicroFit 2x3, J4 JST-GH 4Pin, Q17 NMOS, Q18 NMOS, SW1 SW_DIP_x06, U1 AZ1117H-ADJ, U1 STM32F072RBT6, U3 AZ1117-3.3, U4 W25Q128JVP, U5 MCP2562-E-SN, U6 L7805, U7 L7805, U8 MCP4017-xxxxLT, U9 LM3488MM, Y1 8MHz 12pF

Commit message: updates to the schematics, rough component placement in the PCB layout
Parts:
- removed TP11, TP12, TP5, TP6: TestPoint, TestPoint:TestPoint_Pad_2.0x2.0mm, symbol Connector:TestPoint
- removed U1: STM32F072RBT6, Package_QFP:LQFP-64_10x10mm_P0.5mm, symbol MCU_ST_STM32F0:STM32F072RBTx
- added C1: 100n, Capacitor_SMD:C_0603_1608Metric_Pad1.08x0.95mm_HandSolder, symbol Device:C
- added D17, D18, D19: D_Schottky, Diode_SMD:D_SMA, symbol Device:D_Schottky
- added H1, H2, H3, H4: MountingHole_Pad, MountingHole:MountingHole_3.2mm_M3_Pad_Via, symbol Mechanical:MountingHole_Pad
- added J4 (x2): JST-GH 4Pin, Connector_JST:JST_GH_BM04B-GHS-TBT_1x04-1MP_P1.25mm_Vertical, symbol Connector:Conn_01x04_Pin
- added R18, R19: 10k, Resistor_SMD:R_0603_1608Metric, symbol Device:R_Small
- added R59: 10k, Resistor_SMD:R_0603_1608Metric_Pad0.98x0.95mm_HandSolder, symbol Device:R
- added R62: 5m, Resistor_SMD:R_2512_6332Metric, symbol Device:R
- added TH1: 10k, Resistor_SMD:R_0603_1608Metric_Pad0.98x0.95mm_HandSolder, symbol Device:Thermistor_NTC
- added U10: STM32F103RCTx, Package_QFP:LQFP-64_10x10mm_P0.5mm, symbol MCU_ST_STM32F1:STM32F103RCTx
- added U7: INA213, Package_TO_SOT_SMD:SOT-363_SC-70-6, symbol frodo_power_module:INA210
- C12: value 10u -> 100n; footprint Capacitor_SMD:C_1206_3216Metric_Pad1.33x1.80mm_HandSolder -> Capacitor_SMD:C_0603_1608Metric_Pad1.08x0.95mm_HandSolder
- C12: value 10u -> 330n; footprint Capacitor_SMD:C_1206_3216Metric_Pad1.33x1.80mm_HandSolder -> Capacitor_SMD:C_0603_1608Metric_Pad1.08x0.95mm_HandSolder
- D7, D8: footprint Diode_SMD:D_SOD-123F -> Diode_SMD:D_SMA
- TP1, TP10, TP2, TP3, TP4, TP7, TP8, TP9: footprint TestPoint:TestPoint_Pad_2.0x2.0mm -> TestPoint:TestPoint_Pad_D2.0mm
Connections:
- net USART3_RX is gone; now on net U3_RX-I2C2_SDA: J4.3 (Pin_3)
- net USART3_TX is gone; now on net U3_TX-I2C2_SCL: J4.2 (Pin_2)
- net +3.3V: now also C1.1, R18.2, R59.1, U10.1 (VBAT), U10.19 (VDD), U10.32 (VDD), U10.48 (VDD), U10.64 (VDD), U7.3 (V+)
- net +3.3VA: now also U10.13 (VDDA)
- net +VSW: no longer C12.1, C12.1, C12.1, C12.1, U1.3 (VI), U3.3 (VI), U6.1 (IN), U7.1 (IN)
- net +VSW_fused: now also C12.1, C12.1, C12.1, C12.1, U1.3 (VI), U3.3 (VI), U6.1 (IN), U7.1 (IN), D18.1 (K), D19.1 (K); no longer F1.2
- net BOOTO: now also U10.60 (BOOT0)
- net CAN_RX: now also U10.44 (PA11)
- net CAN_TX: now also U10.45 (PA12)
- net GND: now also C1.2, H1.1, H2.1, H3.1, H4.1, J4.4 (Pin_4), J4.4 (Pin_4), R19.1, TH1.2, U10.12 (VSSA), U10.18 (VSS), U10.31 (VSS), U10.47 (VSS), U10.63 (VSS), U7.2 (GND)
- net HSE_IN: now also U10.5 (PD0)
- net HSE_OUT: now also U10.6 (PD1)
- net NRST: now also U10.7 (NRST)
- net SPI1_MISO: now also U10.56 (PB4)
- net SPI1_MOSI: now also U10.57 (PB5)
- net SPI1_SCK: now also U10.55 (PB3)
- net SPI_CS_FLASH: now also U10.50 (PA15)
- net STAT_LED0: now also U10.33 (PB12)
- net STAT_LED1: now also U10.34 (PB13)
- net STAT_LED2: now also U10.35 (PB14)
- net SW3: now also U10.37 (PC6)
- net SW4: now also U10.38 (PC7)
- net SW5: now also U10.39 (PC8)
- net SWCLK: now also U10.49 (PA14)
- net SWDIO: now also U10.46 (PA13)
- net VCOM: now also J4.1 (Pin_1), J4.1 (Pin_1)
- net VDC_fused: now also D8.1 (K), D17.1 (K); no longer F2.2
- net Vboost: no longer D8.1 (K)
- net Vdrive: now also R62.1, U7.4 (+); no longer JP1.2 (B), JP2.2 (B), JP3.2 (B), JP4.2 (B), JP5.2 (B), JP6.2 (B), JP7.2 (B), JP8.2 (B)
- net at D7.2 (A), L1.2, Q17.1 (D)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: no longer D8.2 (A)
- net SCA renamed U3_RX-I2C2_SDA
- net U3_RX-I2C2_SDA: now also U10.30 (PB11)
- net SCL renamed U3_TX-I2C2_SCL
- net U3_TX-I2C2_SCL: now also U10.29 (PB10)
- net USART1_RX renamed U1_RX-I2C1_SDA
- net U1_RX-I2C1_SDA: now also U10.59 (PB7)
- net USART1_TX renamed U1_TX-I2C1_SCL
- net U1_TX-I2C1_SCL: now also U10.58 (PB6)
- net USART2_RX renamed U2_RX-AIN5
- net U2_RX-AIN5: now also U10.17 (PA3)
- net USART2_TX renamed U2_TX-AIN4
- net U2_TX-AIN4: now also U10.16 (PA2)
- net USART4_RX renamed U4_RX
- net U4_RX: now also U10.52 (PC11)
- net USART4_TX renamed U4_TX
- net U4_TX: now also U10.51 (PC10)
- new net: D17.2 (A), D8.2 (A), F2.2
- new net: R18.1, R19.2, U7.1 (REF)
- new net: D18.2 (A), D19.2 (A), F1.2
- new net AIN0: J4.2 (Pin_2), U10.8 (PC0)
- new net AIN1: J4.3 (Pin_3), U10.9 (PC1)
- new net AIN2: J4.2 (Pin_2), U10.10 (PC2)
- new net AIN3: J4.3 (Pin_3), U10.11 (PC3)
- new net I_sense: U10.27 (PB1), U7.6
- new net TH_sense: R59.2, TH1.1
- new net Vdrive_pre_I_sense: JP1.2 (B), JP2.2 (B), JP3.2 (B), JP4.2 (B), JP5.2 (B), JP6.2 (B), JP7.2 (B), JP8.2 (B), R62.2, U7.5 (-)
- no-connect marks 13 -> 2
Other:
- note added: "Isense"
- note added: "Mounting"
- note added: "Those can be anywhere"
- note added: "Those must be on AINs"
- note added: "Those should be on timers"
- moved on the sheet: C1, C12, C13, C2, C23, C24, C25, C26, C27, C28, C29, C3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
