File: frodo_io_module.kicad_pcb (KiCad board)
At the start: 4 copper layers, 55 x 55 mm, 163 parts, among them J1 Conn_02x04_Top_Bottom, J10 JST-GH 4Pin, J14 USB_C_Receptacle_USB2.0, J16 TC2050, J2 Conn_02x05_Counter_Clockwise, J3 Conn_02x04_Top_Bottom, J4 Conn_02x03_Counter_Clockwise, J5 JST-GH 4Pin, J6 JST-GH 4Pin, J7 JST-GH 4Pin, J8 JST-GH 4Pin, J9 JST-GH 4Pin, Q1 AOSP21321, Q2 AOSP21321, Q3 NMOS, Q4 NMOS, Q5 AOSP21321, Q6 AOSP21321, Q7 NMOS, Q8 NMOS, SW1 KMR721NGLFS, SW2 KMR721NGLFS, SW3 KMR721NGLFS, U1 L7805, U10 INA181A2IDBVT, U11 MCP2562-E-SN, U12 TPD4E1U06, U2 L7805, U3 STM32F105RCTx, U4 AZ1117H-ADJ, U5 AZ1117H-ADJ, U6 INA181, U7 INA181, U8 MCP2562-E-SN, U9 TPD4E1U06, Y1 8MHz 12pF

Commit message: work on usb connector routing
Parts:
- moved D14 164.6 mm to (125.3, 111.7), turned to 90 degrees
- moved C15 125.9 mm to (126.2, 114.7)
- moved C18 122.4 mm to (128.4, 118.0), turned to 180 degrees
- moved C19 121.8 mm to (130.3, 118.0)
- moved C24 117.4 mm to (124.6, 108.8)
- moved SW2 109.0 mm to (131.8, 111.8)
- moved R12 105.3 mm to (128.8, 119.6), turned to 90 degrees
- moved R21 97.1 mm to (123.6, 110.6), turned to 90 degrees
- moved U9 93.0 mm to (127.5, 111.6), turned to 90 degrees
- moved R22 90.1 mm to (126.2, 106.6), turned to 90 degrees
- moved R24 86.7 mm to (123.6, 112.6), turned to 90 degrees
- moved R23 86.1 mm to (129.2, 106.7), turned to 90 degrees
- moved R25 79.0 mm to (127.2, 109.2), turned to -90 degrees
- moved R26 75.6 mm to (128.3, 109.2), turned to 90 degrees
- moved C22 24.9 mm to (92.0, 116.4)
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Routing:
- net NRST: track 0.00 -> 13.0 mm
- net /VBUS: track 0.00 -> 12.8 mm, vias 0 -> 1
- net /D0+: track 0.00 -> 7.62 mm, vias 0 -> 1
- net /D0-: track 0.00 -> 6.72 mm, vias 0 -> 1
- net Net-(D8-A): track 4.36 -> 0.00 mm
- net HSE_IN: track 10.7 -> 7.86 mm
- net GND: track 12.9 -> 10.2 mm
- net Net-(C18-Pad1): track 0.00 -> 2.71 mm
- net Net-(J14-CC2): track 0.00 -> 1.85 mm, vias 0 -> 1
- net Net-(J14-CC1): track 0.00 -> 1.73 mm, vias 0 -> 1
- net HSE_OUT: track 0.00 -> 1.59 mm
- net USB_FS_VBUS: track 0.00 -> 0.97 mm

Commit message: fixed usb, added footprints
Parts:
- removed the C20 at (28.1, 54.4)
- removed the D13 at (265.2, 18.5)
- removed D21, D22, D23, D24: D, Diode_SMD:D_SOD-323_HandSoldering
- removed F4: 10A, Fuse:Fuse_1206_3216Metric
- removed FB14: BLM15PD121SN1D, Inductor_SMD:L_0402_1005Metric
- removed the R16 at (98.5, 34.9)
- removed the R35 at (113.7, 28.7)
- removed Shunt1: 250mR 1%, Resistor_SMD:R_0805_2012Metric
- removed the U7 at (203.2, 122.0)
- added C26: 100n, Capacitor_SMD:C_0402_1005Metric, F.Cu at (80.5, 75.8)
- added D16: D, Diode_SMD:D_SOD-323_HandSoldering, F.Cu at (89.2, 76.3)
- added D17: D, Diode_SMD:D_SOD-323_HandSoldering, F.Cu at (89.2, 79.2)
- added D18: D, Diode_SMD:D_SOD-323_HandSoldering, F.Cu at (89.2, 68.4)
- added D19: D, Diode_SMD:D_SOD-323_HandSoldering, F.Cu at (89.2, 71.3)
- added FB13: BLM15PD121SN1D, Inductor_SMD:L_0402_1005Metric, F.Cu at (77.6, 67.9)
- added J5: Conn_02x04_Odd_Even, Connector_PinHeader_1.27mm:PinHeader_2x04_P1.27mm_Vertical_SMD, B.Cu at (112.0, 108.5)
- added R10: 100, Resistor_SMD:R_0402_1005Metric, F.Cu at (145.9, 71.4)
- added R11: 1k, Resistor_SMD:R_0402_1005Metric, F.Cu at (77.6, 69.9)
- added R12: 100, Resistor_SMD:R_0402_1005Metric, F.Cu at (143.0, 73.4)
- added R13: 100, Resistor_SMD:R_0402_1005Metric, F.Cu at (145.9, 73.4)
- added R14: 1k, Resistor_SMD:R_0402_1005Metric, F.Cu at (77.6, 71.9)
- added R18: 100, Resistor_SMD:R_0402_1005Metric, F.Cu at (143.0, 75.4)
- added R19: 100, Resistor_SMD:R_0402_1005Metric, F.Cu at (145.9, 75.4)
- added R20: 1k, Resistor_SMD:R_0402_1005Metric, F.Cu at (77.6, 73.9)
- added R21: 100, Resistor_SMD:R_0402_1005Metric, F.Cu at (143.0, 77.3)
- added R22: 100, Resistor_SMD:R_0402_1005Metric, F.Cu at (145.9, 77.3)
- added R23: 1k, Resistor_SMD:R_0402_1005Metric, F.Cu at (77.6, 75.9)
- added R27: 25m, Resistor_SMD:R_1206_3216Metric_Pad1.30x1.75mm_HandSolder, F.Cu at (144.6, 83.3)
- added R31: 25m, Resistor_SMD:R_1206_3216Metric_Pad1.30x1.75mm_HandSolder, F.Cu at (144.6, 80.0)
- added R9: 100, Resistor_SMD:R_0402_1005Metric, F.Cu at (143.0, 71.4)
- added U9: INA181A1, Package_TO_SOT_SMD:SOT-23-6, F.Cu at (81.6, 72.6)
- J2: value Conn_02x05_Counter_Clockwise -> Conn_02x10_Odd_Even; footprint Connector_PinHeader_1.27mm:PinHeader_2x04_P1.27mm_Vertical_SMD -> Connector_PinHeader_1.27mm:PinHeader_2x10_P1.27mm_Vertical_SMD
- J4: value Conn_02x03_Counter_Clockwise -> Conn_02x03_Odd_Even
- U12: renamed from U10; value INA181A2IDBVT -> INA181A1
- U6: value INA181 -> W25Q128JVP; footprint Package_TO_SOT_SMD:SOT-23-6 -> Package_SO:SOIC-8_5.3x5.3mm_P1.27mm
- moved U6 227.6 mm to (4.67, 2.92)
- moved F3 137.9 mm to (81.8, 68.6)
- moved H3 7.07 mm to (156.0, 156.0)
- moved J3 5.16 mm to (150.2, 125.4)
- moved J1 5.16 mm to (150.2, 143.6)
- moved H2 5.00 mm to (104.0, 156.0)
- moved H4 5.00 mm to (156.0, 104.0)
- moved J12 4.87 mm to (139.8, 150.0)
- moved J13 4.87 mm to (117.2, 150.0)
- moved J14 4.87 mm to (128.5, 150.0)
- moved J2 3.54 mm to (130.0, 130.0), turned to 0 degrees
- moved C21 3.51 mm to (132.5, 120.8)
- moved C5 3.51 mm to (133.6, 137.4)
- moved C6 3.51 mm to (137.4, 126.2)
- moved R25 3.51 mm to (131.0, 122.3)
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- renumbered C21 to C18, C22 to C19, C18 to C20, C19 to C21, C23 to C22, C24 to C23, C25 to C24, C26 to C25, C30 to C29, C29 to C30, D15 to D13, D16 to D14, D14 to D15, FB13 to FB10, FB6 to FB11, FB10 to FB12, FB3 to FB2, FB7 to FB3, FB11 to FB4, FB4 to FB5, FB8 to FB6, FB12 to FB7, FB5 to FB8, J9 to J10, J10 to J11, J11 to J12, J12 to J13, J15 to J14, J14 to J15, J5 to J6, J6 to J7, J7 to J8, J8 to J9, R15 to R1, R9 to R15, R10 to R16, R52 to R17, R11 to R24, R12 to R25, R14 to R26, R13 to R28, R17 to R29, R53 to R3, R18 to R30, R19 to R32, R20 to R33, R21 to R34, R22 to R35, R23 to R36, R24 to R37, R25 to R38, R26 to R39, R5 to R4, R27 to R40, R28 to R41, R31 to R42, R32 to R43, R33 to R44, R34 to R45, R29 to R46, R30 to R47, R37 to R48, R38 to R49, R6 to R5, R39 to R50, R36 to R51, R40 to R52, R41 to R53, R42 to R54, R43 to R55, R44 to R56, R45 to R57, R46 to R58, R47 to R59, R7 to R6, R48 to R60, R49 to R61, R50 to R62, R51 to R63, R8 to R7, R4 to R8, U11 to U10, U12 to U11, U8 to U7, U9 to U8
Connections:
- D13 pad 2: high_current2 -> SH21
- D14 pad 2: high_current -> SH11
- F1 pad 2: v_main_pre_sense -> main_voltage
- F2 pad 2: high_current -> SH12
- F3 pad 1: high_current -> /Digital Output1/VD
- F3 pad 2: /Digital Output1/VD -> SH22
- FB10 pad 1: AIN2 -> Net-(FB10-Pad1)
- FB11 pad 1: COM2_2 -> Net-(FB11-Pad1)
- FB12 pad 1: CON4_2 -> Net-(FB12-Pad1)
- FB2 pad 1: COM1_1 -> Net-(FB2-Pad1)
- FB3 pad 1: COM3_1 -> Net-(FB3-Pad1)
- FB4 pad 1: AIN0 -> Net-(FB4-Pad1)
- FB5 pad 1: COM1_2 -> Net-(FB5-Pad1)
- FB6 pad 1: COM3_2 -> Net-(FB6-Pad1)
- FB7 pad 1: AIN1 -> Net-(FB7-Pad1)
- FB8 pad 1: COM2_1 -> Net-(FB8-Pad1)
- FB9 pad 1: COM4_1 -> Net-(FB9-Pad1)
- J12 pad 3: high_current -> SH11
- J12 pad 4: high_current2 -> SH21
- J16 pad 6: Net-(J16-Pin_6) -> SWCLK
- J2 pad 1: unconnected-(J2-Pin_1-Pad1) -> +5V
- J2 pad 2: unconnected-(J2-Pin_2-Pad2) -> +5V
- J2 pad 3: unconnected-(J2-Pin_3-Pad3) -> GND
- J2 pad 4: unconnected-(J2-Pin_4-Pad4) -> SPI1_SCK
- J2 pad 5: unconnected-(J2-Pin_5-Pad5) -> IO-0 (UART5 TX)
- J2 pad 6: unconnected-(J2-Pin_6-Pad6) -> SPI1_MISO
- J2 pad 7: unconnected-(J2-Pin_7-Pad7) -> IO-1 (UART5 RX)
- J2 pad 8: unconnected-(J2-Pin_8-Pad8) -> SPI1_MOSI
- J4 pad 2: VS1 -> +3.3V
- J4 pad 3: +5V -> VS1
- J4 pad 4: +5V -> VS2
- J4 pad 5: VS2 -> +5V
- J4 pad 6: +3.3V -> +5V
- R4 pad 2: U1_TX-I2C1_SCL -> Net-(J5-Pin_2)
- R42 pad 1: v_main_pre_sense -> main_voltage
- R43 pad 1: high_current -> SH11
- R44 pad 1: high_current2 -> SH21
- R47 pad 1: Net-(J16-Pin_6) -> SWCLK
- R5 pad 2: U1_RX-I2C1_SDA -> Net-(J5-Pin_4)
- R6 pad 2: U3_TX-I2C2_SCL -> Net-(J5-Pin_6)
- R7 pad 2: U3_RX-I2C2_SDA -> Net-(J5-Pin_8)
- U11 pad 4: Net-(J16-Pin_6) -> SWCLK
- U12 pad 1: I_sense_main -> I_sense_2
- U12 pad 3: v_main_pre_sense -> SH21
- U12 pad 4: main_voltage -> SH22
- U3 pad 2: unconnected-(U3-PC13-Pad2) -> IO-6
- U3 pad 21: unconnected-(U3-PA5-Pad21) -> IO-2 (ADC/DAC)
- U3 pad 22: unconnected-(U3-PA6-Pad22) -> I_sense_1
- U3 pad 23: unconnected-(U3-PA7-Pad23) -> I_sense_2
- U3 pad 28: unconnected-(U3-PB2-Pad28) -> SPI_CS_FLASH
- U3 pad 3: unconnected-(U3-PC14-Pad3) -> IO-7
- U3 pad 35: IO-0 -> IO-4
- U3 pad 36: IO-1 -> IO-5
- U3 pad 37: unconnected-(U3-PC6-Pad37) -> SWITCH
- U3 pad 4: unconnected-(U3-PC15-Pad4) -> IO-8
- U3 pad 42: HC_OUT_2 -> USB_FS_VBUS
- U3 pad 43: IO-2 -> HC_OUT_2
- U3 pad 44: CAN1_RX -> USB_D-
- U3 pad 45: CAN1_TX -> USB_D+
- U3 pad 53: IO-3 (UART5 TX) -> IO-0 (UART5 TX)
- U3 pad 54: IO-4 (UART5 RX) -> IO-1 (UART5 RX)
- U3 pad 58: COM2_1 -> COM1_1
- U3 pad 59: COM2_2 -> COM1_2
- U3 pad 61: SWITCH -> CAN1_RX
- U3 pad 62: SPI_CS_FLASH -> CAN1_TX
- U3 pad 8: I_sense_main -> IO-3 (ADC)
- U6 pad 1: adc_cont_check -> SPI_CS_FLASH
- U6 pad 2: GND -> SPI1_MISO
- U6 pad 3: Net-(U6-+) -> unconnected-(U6-IO2-Pad3)
- U6 pad 4: Net-(D13-A) -> GND
- U6 pad 5: GND -> SPI1_MOSI
- U6 pad 6: +3.3V -> SPI1_SCK
Routing:
- net unconnected-(J15-SBU2-PadB8): track 0.00 -> 3.79 mm
- net /D0+: track 7.62 -> 3.83 mm
- net NRST: track 13.0 -> 11.7 mm
Other:
- board size 55 x 55 mm -> 60 x 60 mm

Commit message: some more changes
Parts:
- added J14: Conn_02x03_Odd_Even, Connector_PinHeader_2.54mm:PinHeader_2x03_P2.54mm_Vertical_SMD, B.Cu at (124.4, 141.0)
- moved J13 11.3 mm to (128.5, 150.0)
- moved J15 11.3 mm to (117.2, 150.0)
- moved J10 0.25 mm to (103.2, 145.0)
- moved J8 0.20 mm to (112.0, 135.0)
- moved J11 0.10 mm to (112.0, 125.0)
- turned J2 to 90 degrees
- renumbered J14 to J15, J15 to J16, J16 to J17
Connections:
- J15 pad 1: /Digital Output1/OUT1 -> GND
- J15 pad 2: /Digital Output1/OUT2 -> GND
- J15 pad 3: GND -> /Digital Output1/OUT2
- J15 pad 4: GND -> /Digital Output1/OUT1
Routing:
- net /D0-: track 6.72 -> 8.54 mm, vias 1 -> 2
- net Net-(J16-CC1): track 1.73 -> 0.00 mm, vias 1 -> 0
- net Net-(J16-CC2): track 1.85 -> 0.76 mm
- net (no net): track 0.00 -> 0.99 mm
Other:
- board text added: "1"
- board text added: "2"
- board text added: "HC in"
- board text added: "gnd"
- board text added: "io/servo"
- board text added: "o1|o2 gnd|gnd"
- board text added: "o1|vcc"
- board text added: "o2|sig"
- board text added: "o3|o4 gnd|gnd"
- board text added: "o3|sig"
- board text added: "o3|vcc"
- board text added: "v2|v1 gnd|gnd"
- board text removed: "COM5"
